File: eagle/main.brd (EAGLE design)
At the start: 98.7 x 90.2 mm, 33 parts, among them IC1 7805TV, U1 INA213AIDCKT, U2 LM1117MP-3.3, U3 INA213AIDCKT, U5 S25FL064K0SMFI011, U6 INA146UA, U7 INA213AIDCKT, U8 INA146UA

Commit message: rename PV, BAT, LOAD signals
Connections:
- net BAT_GND renamed BAT_VN
- net BAT_IN renamed BAT_VPA
- net BAT_OUT renamed BAT_VPB
- net LOAD_GND renamed LOAD_VN
- net LOAD_IN renamed LOAD_VPA
- net LOAD_OUT renamed LOAD_VPB
- net PV_GND renamed PV_VN
- net PV_IN renamed PV_VPA
- net PV_OUT renamed PV_VPB
Changed lines of the file:
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@@
 <contactref element="U$1" pad="VIN"/>
 </signal>
-<signal name="PV_IN">
+<signal name="PV_VPA">
 <contactref element="CON_PV" pad="P$1"/>
 <contactref element="U1" pad="4"/>
@@
 <wire x1="6.35" y1="12.7" x2="20.0914" y2="19.6596" width="0" layer="19" extent="1-1"/>
 </signal>
-<signal name="PV_OUT">
-<contactref element="CON_PV" pad="P$2"/>
-<contactref element="U1" pad="5"/>
-<contactref element="R1" pad="1"/>
-<contactref element="R2" pad="2"/>
-<contactref element="U6" pad="3"/>
-<wire x1="6.35" y1="22.86" x2="-85.0138" y2="-106.045" width="0" layer="19" extent="1-1"/>
-<wire x1="16.25" y1="16.51" x2="6.35" y2="22.86" width="0" layer="19" extent="1-1"/>
-<wire x1="20.0914" y1="20.32" x2="16.25" y2="16.51" width="0" layer="19" extent="1-1"/>
-<wire x1="-60.11" y1="62.23" x2="6.35" y2="22.86" width="0" layer="19" extent="1-1"/>
-</signal>
-<signal name="LOAD_IN">
+<signal name="LOAD_VPA">
 <contactref element="CON_LOAD" pad="P$1"/>
 <contactref element="R4" pad="2"/>
@@
 <wire x1="6.35" y1="38.1" x2="20.0914" y2="45.0596" width="0" layer="19" extent="1-1"/>
 </signal>
-<signal name="LOAD_OUT">
-<contactref element="CON_LOAD" pad="P$2"/>
-<contactref element="R4" pad="1"/>
-<contactref element="U3" pad="5"/>
-<wire x1="16.25" y1="41.91" x2="20.0914" y2="45.72" width="0" layer="19" extent="1-1"/>
-<wire x1="6.35" y1="48.26" x2="16.25" y2="41.91" width="0" layer="19" extent="1-1"/>
-</signal>
-<signal name="BAT_IN">
+<signal name="BAT_VPA">
 <contactref element="CON_BAT" pad="P$1"/>
 <contactref element="R5" pad="2"/>
@@
 <wire x1="22.86" y1="52.07" x2="6.35" y2="63.5" width="0" layer="19" extent="1-1"/>
 </signal>
-<signal name="BAT_OUT">
+<signal name="BAT_VPB">
 <contactref element="CON_BAT" pad="P$2"/>
 <contactref element="R5" pad="1"/>
@@
 <contactref element="U5" pad="2"/>
 </signal>
-<signal name="LOAD_GND">
+<signal name="LOAD_VN">
 <contactref element="CON_LOAD" pad="P$3"/>
 <contactref element="CON_LOAD" pad="P$4"/>
 <wire x1="6.35" y1="43.18" x2="6.35" y2="53.34" width="0" layer="19" extent="1-1"/>
 </signal>
-<signal name="PV_GND">
+<signal name="PV_VN">
 <contactref element="CON_PV" pad="P$3"/>
 <contactref element="CON_PV" pad="P$4"/>
@@
 <wire x1="-85.0138" y1="-130.175" x2="-86.78" y2="-157.48" width="0" layer="19" extent="1-1"/>
 </signal>
-<signal name="BAT_GND">
+<signal name="BAT_VN">
 <contactref element="CON_BAT" pad="P$3"/>
 <contactref element="CON_BAT" pad="P$4"/>
@@
 <contactref element="CON_GPIO" pad="9"/>
 </signal>
+<signal name="PV_VPB">
+<contactref element="CON_PV" pad="P$2"/>
+<contactref element="U1" pad="5"/>
+<contactref element="R1" pad="1"/>
+<contactref element="R2" pad="2"/>
+<contactref element="U6" pad="3"/>
+<wire x1="6.35" y1="22.86" x2="-85.0138" y2="-106.045" width="0" layer="19" extent="1-1"/>
+<wire x1="16.25" y1="16.51" x2="6.35" y2="22.86" width="0" layer="19" extent="1-1"/>
+<wire x1="20.0914" y1="20.32" x2="16.25" y2="16.51" width="0" layer="19" extent="1-1"/>
+<wire x1="-60.11" y1="62.23" x2="6.35" y2="22.86" width="0" layer="19" extent="1-1"/>
+</signal>
+<signal name="LOAD_VPB">
+<contactref element="CON_LOAD" pad="P$2"/>
+<contactref element="R4" pad="1"/>
+<contactref element="U3" pad="5"/>
+<wire x1="16.25" y1="41.91" x2="20.0914" y2="45.72" width="0" layer="19" extent="1-1"/>
+<wire x1="6.35" y1="48.26" x2="16.25" y2="41.91" width="0" layer="19" extent="1-1"/>
+</signal>
 </signals>
